File: hardware/robo_board/robo_board.sch (KiCad schematic (older format))
At the start: 28 parts, among them J101 Conn_01x03_Female, J102 Conn_01x06_Female, Q101 Q_Photo_NPN, Q102 Q_Photo_NPN, Q103 Q_Photo_NPN, Q104 Q_Photo_NPN, Q105 Q_Photo_NPN, Q106 Q_Photo_NPN, SW101 SW_Push, SW102 SW_Push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

Commit message: Add battery power to robo_board scheme
Parts:
- added BT101: 3V, symbol Device:Battery
- added SW103: SW_SPST, symbol Switch:SW_SPST
Connections:
- net Vdrive is gone; now on net VDD: C103.1, C104.1, U102.16 (VCC1), U102.8 (VCC2)
- net GND: now also BT101.2 (-)
- net VDD: now also SW103.2 (B)
- new net: BT101.1 (+), SW103.1 (A)
Changed lines of the file:
@@
 Wire Wire Line
 	5650 2600 5200 2600
-Wire Bus Line
-	600  4950 600  7550
-Wire Bus Line
-	2650 5000 2650 7550
-Wire Bus Line
-	5100 4800 5100 7550
-Wire Bus Line
-	5900 2200 5900 4800
-Wire Bus Line
-	5100 2150 5100 4800
 Text Label 5250 2300 0    50   ~ 0
 BLUE
@@
 Text Label 4850 4350 0    50   ~ 0
 R2
+$Comp
+L Device:Battery BT101
+U 1 1 5E78D938
+P 1700 3100
+F 0 "BT101" H 1808 3146 50  0000 L CNN
+F 1 "3V" H 1808 3055 50  0000 L CNN
+F 2 "" V 1700 3160 50  0001 C CNN
+F 3 "~" V 1700 3160 50  0001 C CNN
+	1    1700 3100
+	1    0    0    -1
+$EndComp
+$Comp
+L power:GND #PWR?
+U 1 1 5E78F166
+P 1700 3500
+F 0 "#PWR?" H 1700 3250 50  0001 C CNN
+F 1 "GND" H 1705 3327 50  0000 C CNN
+F 2 "" H 1700 3500 50  0001 C CNN
+F 3 "" H 1700 3500 50  0001 C CNN
+	1    1700 3500
+	1    0    0    -1
+$EndComp
+Wire Wire Line
+	1700 3300 1700 3500
+$Comp
+L power:VDD #PWR?
+U 1 1 5E797467
+P 1450 2100
+F 0 "#PWR?" H 1450 1950 50  0001 C CNN
+F 1 "VDD" H 1467 2273 50  0000 C CNN
+F 2 "" H 1450 2100 50  0001 C CNN
+F 3 "" H 1450 2100 50  0001 C CNN
+	1    1450 2100
+	1    0    0    -1
+$EndComp
+$Comp
+L power:Vdrive #PWR?
+U 1 1 5E797EE3
+P 1900 2100
+F 0 "#PWR?" H 1700 1950 50  0001 C CNN
+F 1 "Vdrive" H 1917 2273 50  0000 C CNN
+F 2 "" H 1900 2100 50  0001 C CNN
+F 3 "" H 1900 2100 50  0001 C CNN
+	1    1900 2100
+	1    0    0    -1
+$EndComp
+$Comp
+L Switch:SW_SPST SW103
+U 1 1 5E7995B1
+P 1700 2550
+F 0 "SW103" V 1746 2462 50  0000 R CNN
+F 1 "SW_SPST" V 1655 2462 50  0000 R CNN
+F 2 "" H 1700 2550 50  0001 C CNN
+F 3 "~" H 1700 2550 50  0001 C CNN
+	1    1700 2550
+	0    -1   -1   0
+$EndComp
+Wire Wire Line
+	1700 2350 1700 2150
+Wire Wire Line
+	1700 2150 1450 2150
+Wire Wire Line
+	1450 2150 1450 2100
+Wire Wire Line
+	1700 2150 1900 2150
+Wire Wire Line
+	1900 2150 1900 2100
+Connection ~ 1700 2150
+Wire Wire Line
+	1700 2750 1700 2900
+Wire Bus Line
+	600  4950 600  7550
+Wire Bus Line
+	2650 5000 2650 7550
+Wire Bus Line
+	5100 4800 5100 7550
+Wire Bus Line
+	5900 2200 5900 4800
+Wire Bus Line
+	5100 2150 5100 4800
 $EndSCHEMATC

Commit message: Change photo sensor resistors from 10k to 47k for improve sense
Parts:
- R101, R102, R103, R104, R105, R106: value 10k -> 47k
Changed lines of the file:
@@
 P 1150 5550
 F 0 "R104" H 1220 5596 50  0000 L CNN
-F 1 "10k" H 1220 5505 50  0000 L CNN
+F 1 "47k" H 1220 5505 50  0000 L CNN
 F 2 "" V 1080 5550 50  0001 C CNN
 F 3 "~" H 1150 5550 50  0001 C CNN
@@
 P 1800 6100
 F 0 "R106" H 1870 6146 50  0000 L CNN
-F 1 "10k" H 1870 6055 50  0000 L CNN
+F 1 "47k" H 1870 6055 50  0000 L CNN
 F 2 "" V 1730 6100 50  0001 C CNN
 F 3 "~" H 1800 6100 50  0001 C CNN
@@
 P 3250 5500
 F 0 "R101" H 3320 5546 50  0000 L CNN
-F 1 "10k" H 3320 5455 50  0000 L CNN
+F 1 "47k" H 3320 5455 50  0000 L CNN
 F 2 "" V 3180 5500 50  0001 C CNN
 F 3 "~" H 3250 5500 50  0001 C CNN
@@
 P 3600 5800
 F 0 "R102" H 3670 5846 50  0000 L CNN
-F 1 "10k" H 3670 5755 50  0000 L CNN
+F 1 "47k" H 3670 5755 50  0000 L CNN
 F 2 "" V 3530 5800 50  0001 C CNN
 F 3 "~" H 3600 5800 50  0001 C CNN
@@
 P 3950 6100
 F 0 "R103" H 4020 6146 50  0000 L CNN
-F 1 "10k" H 4020 6055 50  0000 L CNN
+F 1 "47k" H 4020 6055 50  0000 L CNN
 F 2 "" V 3880 6100 50  0001 C CNN
 F 3 "~" H 3950 6100 50  0001 C CNN
@@
 P 1450 5800
 F 0 "R105" H 1520 5846 50  0000 L CNN
-F 1 "10k" H 1520 5755 50  0000 L CNN
+F 1 "47k" H 1520 5755 50  0000 L CNN
 F 2 "" V 1380 5800 50  0001 C CNN
 F 3 "~" H 1450 5800 50  0001 C CNN

Commit message: Add resistor to reset line to avoid signal interference
Parts:
- added R110: 4.7k, symbol Device:R
Connections:
- net RESET: now also R110.2; no longer SW101.1
- new net: R110.1, SW101.1
Changed lines of the file:
@@
 	5900 3850 6000 3950
-Wire Wire Line
-	7300 4000 6000 4000
 Wire Wire Line
 	6000 4000 6000 3950
@@
 Wire Wire Line
 	1700 2750 1700 2900
+$Comp
+L Device:R R110
+U 1 1 5E7BC377
+P 7000 4000
+F 0 "R110" V 6793 4000 50  0000 C CNN
+F 1 "4.7k" V 6884 4000 50  0000 C CNN
+F 2 "" V 6930 4000 50  0001 C CNN
+F 3 "~" H 7000 4000 50  0001 C CNN
+	1    7000 4000
+	0    1    1    0
+$EndComp
+Wire Wire Line
+	7300 4000 7150 4000
+Wire Wire Line
+	6850 4000 6000 4000
 Wire Bus Line
 	600  4950 600  7550

Commit message: Replase wire to N/C for PD7 pin
Connections:
- no-connect marks 0 -> 1
Changed lines of the file:
@@
 Entry Wire Line
 	5000 4550 5100 4650
-Entry Wire Line
-	5000 4650 5100 4750
 Wire Wire Line
 	4800 2250 5000 2250
@@
 Wire Wire Line
 	4800 4550 5000 4550
-Wire Wire Line
-	4800 4650 5000 4650
 Entry Wire Line
 	5900 4250 6000 4350
@@
 Wire Wire Line
 	6850 4000 6000 4000
+NoConn ~ 4800 4650
 Wire Bus Line
 	600  4950 600  7550

Commit message: Change resistor value from 470 to 510 Omh for RGB led
Parts:
- R107, R108, R109: value 470 -> 510
Changed lines of the file:
@@
 P 5850 1700
 F 0 "R109" H 5920 1746 50  0000 L CNN
-F 1 "470" H 5920 1655 50  0000 L CNN
+F 1 "510" H 5920 1655 50  0000 L CNN
 F 2 "" V 5780 1700 50  0001 C CNN
 F 3 "~" H 5850 1700 50  0001 C CNN
@@
 P 5650 1500
 F 0 "R108" H 5720 1546 50  0000 L CNN
-F 1 "470" H 5720 1455 50  0000 L CNN
+F 1 "510" H 5720 1455 50  0000 L CNN
 F 2 "" V 5580 1500 50  0001 C CNN
 F 3 "~" H 5650 1500 50  0001 C CNN
@@
 P 5500 1200
 F 0 "R107" H 5570 1246 50  0000 L CNN
-F 1 "470" H 5570 1155 50  0000 L CNN
+F 1 "510" H 5570 1155 50  0000 L CNN
 F 2 "" V 5430 1200 50  0001 C CNN
 F 3 "~" H 5500 1200 50  0001 C CNN
